File: Projet/Base_Projet_ELN3_2021/Base_Projet_ELN3.sch (KiCad schematic (older format))
At the start: 14 parts

Commit message: Projet quasi fini
Parts:
- added U? (x5): 74HC573, symbol 00_ELN3_Symbols:74HC573
- added U?: 74HC238, symbol 74xx_IEEE:74HC238
- added U? (x5): 4081, symbol 4xxx:4081
- added U? (x2): 74AHC04, symbol 74xx:74AHC04
- added U?: 4072, symbol 4xxx:4072
- P?: symbol Modules_CPE:Mapping_Mémoire_64Ko_XDATA_V2 -> Base_Projet_ELN3-rescue:Mapping_Mémoire_64Ko_XDATA_V2-Modules_CPE
Connections:
- net labels added: +3.3V, 4000H, 8000H, BP_Al, C000H, GND, IR1, IR2, IR3, IR4, RD, WR
- wire segments 24 -> 182
Other:
- note added: "/LD"
- note added: "BP_AL"
- note added: "Bloc Sélection Adresse mémoire"
- note added: "C0"
- note added: "C1"
- note added: "C2"
- note added: "C3"
- note added: "C4"
- note added: "C5"
- note added: "CLK"
- note added: "DCP"
- note added: "DP_IN"
- note added: "DP_OUT"
- note added: "IR1"
- note added: "IR2"
- note added: "IR3"
- note added: "IR4"
- note added: "Registre AFF"
- note added: "Registre GCA"
- note added: "Registre GCP"
- note added: "Registre GDD"
- note added: "Registre MISC"
